File: src/pcb/MicBoard/MicBoard.kicad_pcb (KiCad board)
At the start: 2 copper layers, 1 part

Commit message: added footprints very painfully
Parts:
- added C1: 1uF, PCM_JLCPCB:C_0603, F.Cu at (157.2, 67.2)
- added C2: 100nF, PCM_JLCPCB:C_0603, F.Cu at (157.2, 69.5)
- added J1: Conn_01x10_Pin, F0502-B-10-10G-R:FPC-SMD_F0502-B-10-10G-R, F.Cu at (161.5, 76.0)
- MK1: value IM73D122V01XTMA1 -> IM69D120

Commit message: layout 1 completed
Parts:
- added REF**: MountingHole_3.2mm_M3, MountingHole:MountingHole_3.2mm_M3, F.Cu at (161.5, 69.0)
- moved C2 8.81 mm to (158.5, 60.8), turned to -90 degrees
- moved MK1 7.82 mm to (161.3, 61.8), turned to 90 degrees
- moved C1 3.70 mm to (158.5, 63.8), turned to 90 degrees
Connections:
- J1 pad 1: 3P3 -> GND
- J1 pad 10: GND -> 3P3
- J1 pad 2: DATA -> unconnected-(J1-Pin_2-Pad2)
- J1 pad 3: CLK -> unconnected-(J1-Pin_3-Pad3)
- J1 pad 4: SEL -> unconnected-(J1-Pin_4-Pad4)
- J1 pad 7: unconnected-(J1-Pin_7-Pad7) -> SEL
- J1 pad 8: unconnected-(J1-Pin_8-Pad8) -> CLK
- J1 pad 9: unconnected-(J1-Pin_9-Pad9) -> DATA
Routing:
- net 3P3: track 0.00 -> 16.7 mm
- net SEL: track 0.00 -> 14.0 mm
- net CLK: track 0.00 -> 12.7 mm
- net DATA: track 0.00 -> 12.3 mm

Commit message: finalized lyout for microphone
Parts:
- added C3: TestPoint, TestPoint:TestPoint_THTPad_D1.0mm_Drill0.5mm, F.Cu at (165.5, 63.0)
- added D1: TestPoint, TestPoint:TestPoint_THTPad_D1.0mm_Drill0.5mm, F.Cu at (165.5, 65.0)
- added G1: TestPoint, TestPoint:TestPoint_THTPad_D1.0mm_Drill0.5mm, F.Cu at (165.5, 71.0)
- added S1: TestPoint, TestPoint:TestPoint_THTPad_D1.0mm_Drill0.5mm, F.Cu at (165.5, 67.0)
- added V1: TestPoint, TestPoint:TestPoint_THTPad_D1.0mm_Drill0.5mm, F.Cu at (165.5, 61.0)
- moved C1 1.22 mm to (158.5, 65.0)
- moved C2 1.22 mm to (158.5, 62.0)
- moved MK1 1.11 mm to (161.5, 62.9)
Connections:
- J1 pad 8: CLK -> DATA
- J1 pad 9: DATA -> CLK
Routing:
- net SEL: track 14.0 -> 12.8 mm
- net 3P3: track 16.7 -> 15.9 mm
- net DATA: track 12.3 -> 11.5 mm
- net CLK: track 12.7 -> 13.0 mm, vias 0 -> 2
Other:
- board outline added: 10 x 18.5 mm
