File: src/pcb/MicBoard/MicBoard.kicad_sch (KiCad schematic)
At the start: 1 part

Commit message: first schematic? maybe
Parts:
- removed MK1: IM73A135V01, Sensor_Audio:Infineon_PG-LLGA-5-2, symbol Sensor_Audio:IM73A135V01
- added C1: 100nF, symbol Device:C
- added C2: 1uF, symbol Device:C
- added J1: Conn_01x10_Pin, symbol Connector:Conn_01x10_Pin
- added MK1: IM69D120, Sensor_Audio:Infineon_PG-LLGA-5-1, symbol Sensor_Audio:IM69D120
Connections:
- new net 3P3: C1.1, C2.1, J1.1 (Pin_1), MK1.2 (VDD)
- new net CLK: J1.3 (Pin_3), MK1.3 (CLOCK)
- new net DATA: J1.2 (Pin_2), MK1.1 (DATA)
- new net GND: C1.2, C2.2, J1.10 (Pin_10), MK1.5 (GND)
- new net SEL: J1.4 (Pin_4), MK1.4 (SELECT)
- no-connect marks 0 -> 5
Other:
- company: (none) -> Armaan Gomes
- title: (none) -> Tiny Mic Board

Commit message: added footprints very painfully
Parts:
- removed C1: 100nF, symbol Device:C
- removed C2: 1uF, symbol Device:C
- added C1: 1uF, PCM_JLCPCB:C_0603, symbol PCM_JLCPCB-Capacitors:0603,1uF
- added C2: 100nF, PCM_JLCPCB:C_0603, symbol PCM_JLCPCB-Capacitors:0603,100nF
- J1: footprint (none) -> F0502-B-10-10G-R:FPC-SMD_F0502-B-10-10G-R
Connections:
- net 3P3: now also C1.1, C2.1
- net GND: now also C1.2, C2.2

Commit message: layout 1 completed
Connections:
- net 3P3: now also J1.10 (Pin_10); no longer J1.1 (Pin_1)
- net CLK: now also J1.8 (Pin_8); no longer J1.3 (Pin_3)
- net DATA: now also J1.9 (Pin_9); no longer J1.2 (Pin_2)
- net GND: now also J1.1 (Pin_1); no longer J1.10 (Pin_10)
- net SEL: now also J1.7 (Pin_7); no longer J1.4 (Pin_4)
Other:
- moved on the sheet: J1
Changed lines of the file:
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@@
 	)
 	(no_connect
-		(at 133.35 144.78)
+		(at 130.81 142.24)
 	)
 	(no_connect
-		(at 130.81 144.78)
+		(at 135.89 142.24)
 	)
 	(no_connect
-		(at 138.43 144.78)
+		(at 133.35 142.24)
 	)
 	(no_connect
-		(at 135.89 144.78)
+		(at 140.97 142.24)
 	)
 	(no_connect
-		(at 140.97 144.78)
+		(at 138.43 142.24)
+	)
+	(wire
+		(pts
+			(xy 128.27 139.7) (xy 128.27 142.24)
+		)
+		(stroke
+			(width 0)
+			(type default)
+		)
 	)
 	(wire
@@
 	(wire
 		(pts
-			(xy 128.27 139.7) (xy 128.27 144.78)
-		)
-		(stroke
-			(width 0)
-			(type default)
-		)
-	)
-	(wire
-		(pts
 			(xy 152.4 106.68) (xy 162.56 106.68)
 		)
@@
 	(wire
 		(pts
-			(xy 120.65 139.7) (xy 120.65 144.78)
-		)
-		(stroke
-			(width 0)
-			(type default)
-		)
-	)
-	(wire
-		(pts
 			(xy 138.43 102.87) (xy 138.43 106.68)
 		)
@@
 	(wire
 		(pts
-			(xy 123.19 139.7) (xy 123.19 144.78)
-		)
-		(stroke
-			(width 0)
-			(type default)
-		)
-	)
-	(wire
-		(pts
 			(xy 132.08 116.84) (xy 132.08 121.92)
 		)
@@
 	(wire
 		(pts
-			(xy 125.73 139.7) (xy 125.73 144.78)
-		)
-		(stroke
-			(width 0)
-			(type default)
-		)
-	)
-	(wire
-		(pts
 			(xy 138.43 106.68) (xy 152.4 106.68)
 		)
@@
 	(wire
 		(pts
+			(xy 120.65 139.7) (xy 120.65 142.24)
+		)
+		(stroke
+			(width 0)
+			(type default)
+		)
+	)
+	(wire
+		(pts
+			(xy 143.51 139.7) (xy 143.51 142.24)
+		)
+		(stroke
+			(width 0)
+			(type default)
+		)
+	)
+	(wire
+		(pts
+			(xy 123.19 139.7) (xy 123.19 142.24)
+		)
+		(stroke
+			(width 0)
+			(type default)
+		)
+	)
+	(wire
+		(pts
 			(xy 118.11 106.68) (xy 118.11 114.3)
 		)
@@
 	(wire
 		(pts
-			(xy 143.51 139.7) (xy 143.51 144.78)
+			(xy 125.73 139.7) (xy 125.73 142.24)
 		)
 		(stroke
@@
 	(symbol
 		(lib_id "Connector:Conn_01x10_Pin")
-		(at 130.81 149.86 90)
+		(at 133.35 147.32 270)
+		(mirror x)
 		(unit 1)
 		(exclude_from_sim no)
@@
 		(on_board yes)
 		(dnp no)
-		(fields_autoplaced yes)
 		(property "Reference" "J1"
+			(at 132.08 149.86 90)
+			(effects
+				(font
+					(size 1.27 1.27)
+				)
+			)
+		)
+		(property "Value" "Conn_01x10_Pin"
 			(at 132.08 152.4 90)
 			(effects
@@
 			)
 		)
-		(property "Value" "Conn_01x10_Pin"
-			(at 132.08 154.94 90)
-			(effects
-				(font
-					(size 1.27 1.27)
-				)
-			)
-		)
 		(property "Footprint" "F0502-B-10-10G-R:FPC-SMD_F0502-B-10-10G-R"
-			(at 130.81 149.86 0)
+			(at 133.35 147.32 0)
 			(effects
 				(font
@@
 		)
 		(property "Datasheet" "~"
-			(at 130.81 149.86 0)
+			(at 133.35 147.32 0)
 			(effects
 				(font
@@
 		)
 		(property "Description" "Generic connector, single row, 01x10, script generated"
-			(at 130.81 149.86 0)
-			(effects
-				(font
+			(at 133.35 147.32 0)
+			(effects
+				(font

Commit message: finalized lyout for microphone
Parts:
- added TP1, TP2, TP3, TP4, TP5: TestPoint, TestPoint:TestPoint_THTPad_D1.0mm_Drill0.5mm, symbol Connector:TestPoint
Connections:
- net 3P3: now also TP2.1
- net CLK: now also J1.9 (Pin_9), TP3.1; no longer J1.8 (Pin_8)
- net DATA: now also J1.8 (Pin_8), TP4.1; no longer J1.9 (Pin_9)
- net GND: now also TP1.1
- net SEL: now also TP5.1

Commit message: schematic for lr connector
Parts:
- renumbered TP3 to C3, TP4 to D1, TP1 to G1, TP5 to S1, TP2 to V1
Changed lines of the file:
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@@
 		(dnp no)
 		(fields_autoplaced yes)
-		(property "Reference" "TP2"
+		(property "Reference" "V1"
 			(at 170.18 128.7779 0)
 			(effects
@@
 			(project "MicBoard"
 				(path "/2461514a-e2cb-40a8-b313-68e2705f4701"
-					(reference "TP2")
+					(reference "V1")
 					(unit 1)
 				)
@@
 		(dnp no)
 		(fields_autoplaced yes)
-		(property "Reference" "TP4"
+		(property "Reference" "D1"
 			(at 158.75 141.4779 0)
 			(effects
@@
 			(project "MicBoard"
 				(path "/2461514a-e2cb-40a8-b313-68e2705f4701"
-					(reference "TP4")
+					(reference "D1")
 					(unit 1)
 				)
@@
 		(dnp no)
 		(fields_autoplaced yes)
-		(property "Reference" "TP3"
+		(property "Reference" "C3"
 			(at 182.88 128.7779 0)
 			(effects
@@
 			(project "MicBoard"
 				(path "/2461514a-e2cb-40a8-b313-68e2705f4701"
-					(reference "TP3")
+					(reference "C3")
 					(unit 1)
 				)
@@
 		(dnp no)
 		(fields_autoplaced yes)
-		(property "Reference" "TP5"
+		(property "Reference" "S1"
 			(at 170.18 141.4779 0)
 			(effects
@@
 			(project "MicBoard"
 				(path "/2461514a-e2cb-40a8-b313-68e2705f4701"
-					(reference "TP5")
+					(reference "S1")
 					(unit 1)
 				)
@@
 		(dnp no)
 		(fields_autoplaced yes)
-		(property "Reference" "TP1"
+		(property "Reference" "G1"
 			(at 157.48 128.7779 0)
 			(effects
@@
 			(project ""
 				(path "/2461514a-e2cb-40a8-b313-68e2705f4701"
-					(reference "TP1")
+					(reference "G1")
 					(unit 1)
 				)
