File: src/pcb/LRConnectorBoard/LRConnectorBoard.kicad_sch (KiCad schematic)
At the start: 14 parts, among them J1 Conn_01x10_Pin, J2 Conn_01x10_Pin, J3 Conn_01x10_Pin, J4 Conn_01x10_Pin, U1 DS90LV012ATMF/NOPB, U2 DS90LV011ATMF/NOPB, U3 SN74LVC1G17DBVR

Commit message: routed the lr connector
Parts:
- J1, J2, J3, J4: footprint (none) -> F0502-B-10-10G-R:FPC-SMD_F0502-B-10-10G-R
Changed lines of the file:
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@@
 			)
 		)
-		(property "Footprint" ""
+		(property "Footprint" "F0502-B-10-10G-R:FPC-SMD_F0502-B-10-10G-R"
 			(at 232.41 129.54 0)
 			(effects
@@
 			)
 		)
-		(property "Footprint" ""
+		(property "Footprint" "F0502-B-10-10G-R:FPC-SMD_F0502-B-10-10G-R"
 			(at 57.15 127 0)
 			(effects
@@
 			)
 		)
-		(property "Footprint" ""
+		(property "Footprint" "F0502-B-10-10G-R:FPC-SMD_F0502-B-10-10G-R"
 			(at 36.83 40.64 0)
 			(effects
@@
 			)
 		)
-		(property "Footprint" ""
+		(property "Footprint" "F0502-B-10-10G-R:FPC-SMD_F0502-B-10-10G-R"
 			(at 228.6 43.18 0)
 			(effects
